Commit message: prep 2 for moveit setup;

File: src/marv_description/urdf/marv.xacro (robot description, xacro)
@@ -6,4 +6,5 @@
     <xacro:property name="link_width" value="0.1"/>
     <xacro:property name="mass" value="1.0"/>
+    <xacro:property name="gap" value="0.05"/>  <!-- Offset to prevent touching -->
     <!-- Link 1 -->
     <link name="link1">
@@ -33,7 +34,7 @@
         <parent link="link1"/>
         <child link="link2"/>
-        <origin xyz="0 0 ${link1_length}"/>
+        <origin xyz="0 0 ${link1_length + gap}"/>  <!-- Offset added -->
         <axis xyz="1 0 0"/>
-        <limit effort="10.0" lower="-1.57" upper="1.57" velocity="1.0"/>
+        <limit effort="10.0" lower="-3.14" upper="3.14" velocity="1.0"/>
         <dynamics damping="0.5" friction="0.1"/>
     </joint>

File: src/marv_description/urdf/marv.xacro.urdf (robot description, URDF)
Before this commit: robot marv, 2 links, 1 joints
Joints:
- joint joint1: limit lower=-1.57 upper=1.57 effort=10.0 velocity=1.0 -> lower=-3.14 upper=3.14 effort=10.0 velocity=1.0; origin xyz=0 0 1.0 -> xyz=0 0 1.05
